File: PCB/virtualpet.kicad_pcb (KiCad board)
At the start: 2 copper layers, 50 x 90 mm, 5 parts, among them J1 PPTC041LFBN-RC, SW1 SW_Push, SW2 SW_Push, SW3 SW_Push, U1 XIAO-ESP32-C3-DIP

Commit message: BOM + Updated CAD & PCB
Other:
- board text added: "Luis V"
